Commit message: adding iiwa7 + added passive controller lib

File: agx_dual_arm/urdf/iiwa7.urdf (robot description, URDF)
Before this commit: robot iiwa14, 12 links, 11 joints
Links:
- removed link iiwa_link_FTS
- link iiwa_link_0: geometry collision mesh filename=meshes_gazebo/iiwa7/collision/link_0.stl; visual mesh filename=meshes_gazebo/iiwa7/visual/link_0.stl
- link iiwa_link_1: mass 4 -> 3.4525; geometry collision mesh filename=meshes_gazebo/iiwa7/collision/link_1.stl; visual mesh filename=meshes_gazebo/iiwa7/visual/link_1.stl
- link iiwa_link_2: mass 4 -> 3.4821; geometry collision mesh filename=meshes_gazebo/iiwa7/collision/link_2.stl; visual mesh filename=meshes_gazebo/iiwa7/visual/link_2.stl
- link iiwa_link_3: mass 3 -> 4.05623; geometry collision mesh filename=meshes_gazebo/iiwa7/collision/link_3.stl; visual mesh filename=meshes_gazebo/iiwa7/visual/link_3.stl
- link iiwa_link_4: mass 2.7 -> 3.4822; geometry collision mesh filename=meshes_gazebo/iiwa7/collision/link_4.stl; visual mesh filename=meshes_gazebo/iiwa7/visual/link_4.stl
- link iiwa_link_5: mass 1.7 -> 2.1633; geometry collision mesh filename=meshes_gazebo/iiwa7/collision/link_5.stl; visual mesh filename=meshes_gazebo/iiwa7/visual/link_5.stl
- link iiwa_link_6: mass 1.8 -> 2.3466; geometry collision mesh filename=meshes_gazebo/iiwa7/collision/link_6.stl; visual mesh filename=meshes_gazebo/iiwa7/visual/link_6.stl
- link iiwa_link_7: mass 0.3 -> 3.129; geometry collision mesh filename=meshes_gazebo/iiwa7/collision/link_7.stl; visual mesh filename=meshes_gazebo/iiwa7/visual/link_7.stl
- link iiwa_link_grabber: geometry collision mesh filename=meshes_gazebo/force_sensor/meshes/collision/grabber.stl; visual mesh filename=meshes_gazebo/force_sensor/meshes/visual/grabber.stl
Joints:
- removed joint iiwa_joint_FTS
- joint iiwa_joint_1: limit lower=-2.9670597283903604 upper=2.9670597283903604 effort=320 velocity=1.4835298641951802 -> lower=-2.96705972839 upper=2.96705972839 effort=176 velocity=1.71042266695; origin xyz=0 0 0.1575 rpy=0 0 0 -> xyz=0 0 0.15 rpy=0 0 0
- joint iiwa_joint_2: limit lower=-2.0943951023931953 upper=2.0943951023931953 effort=320 velocity=1.4835298641951802 -> lower=-2.09439510239 upper=2.09439510239 effort=176 velocity=1.71042266695; origin xyz=0 0 0.2025 rpy=1.5707963267948966   0 3.141592653589793 -> xyz=0 0 0.19 rpy=1.57079632679   0 3.14159265359
- joint iiwa_joint_3: limit lower=-2.9670597283903604 upper=2.9670597283903604 effort=176 velocity=1.7453292519943295 -> lower=-2.96705972839 upper=2.96705972839 effort=110 velocity=1.74532925199; origin xyz=0 0.2045 0 rpy=1.5707963267948966 0 3.141592653589793 -> xyz=0 0.21 0 rpy=1.57079632679 0 3.14159265359
- joint iiwa_joint_4: limit lower=-2.0943951023931953 upper=2.0943951023931953 effort=176 velocity=1.3089969389957472 -> lower=-2.09439510239 upper=2.09439510239 effort=110 velocity=2.26892802759; origin xyz=0 0 0.2155 rpy=1.5707963267948966 0 0 -> xyz=0 0 0.19 rpy=1.57079632679 0 0
- joint iiwa_joint_5: limit lower=-2.9670597283903604 upper=2.9670597283903604 effort=110 velocity=2.2689280275926285 -> lower=-2.96705972839 upper=2.96705972839 effort=110 velocity=2.44346095279; origin xyz=0 0.1845 0 rpy=-1.5707963267948966 3.141592653589793 0 -> xyz=0 0.21 0 rpy=-1.57079632679 3.14159265359 0
- joint iiwa_joint_6: limit lower=-2.0943951023931953 upper=2.0943951023931953 effort=40 velocity=2.356194490192345 -> lower=-2.09439510239 upper=2.09439510239 effort=40 velocity=3.14159265359; origin xyz=0 0 0.2155 rpy=1.5707963267948966 0 0 -> xyz=0 0.06070 0.19 rpy=1.57079632679 0 0
- joint iiwa_joint_7: limit lower=-3.0543261909900763 upper=3.0543261909900763 effort=40 velocity=2.356194490192345 -> lower=-3.05432619099 upper=3.05432619099 effort=40 velocity=3.14159265359; origin xyz=0 0.081 0 rpy=-1.5707963267948966 3.141592653589793 0 -> xyz=0 0.081 0.06070 rpy=-1.57079632679 3.14159265359 0
- joint iiwa_joint_grabber: origin xyz=0 0 0.0212 rpy=0 0 0 -> xyz=0 0 0.045 rpy=0 0 0; parent iiwa_link_FTS -> iiwa_link_7
